File: PCB/PCB.kicad_pcb (KiCad board)
At the start: 2 copper layers, 68.6 x 81.3 mm, 29 parts, among them J1 Conn_01x14_Socket, J2 Conn_01x08_Socket, J3 Conn_01x08_Socket, J4 Conn_01x02_Socket, J5 Conn_01x08_Socket, SW1 SW_SPDT, U1 Pico, U2 Mini360

Commit message: updated to use internal pull down resistors, remove them from PCB design
Parts:
- removed R10, R11, R12, R13, R14, R15, R16, R9: R, Resistor_SMD:R_0805_2012Metric
Routing:
- net /input 26: track 48.6 -> 29.6 mm
- net /input 21: track 50.3 -> 31.3 mm
- net /input 19: track 50.3 -> 31.3 mm
- net /input 17: track 51.3 -> 32.5 mm
- net /input 20: track 45.0 -> 31.3 mm
- net /input 22: track 43.1 -> 30.3 mm
- net /input 18: track 44.2 -> 31.4 mm
- net /input 16: track 45.2 -> 33.9 mm, vias 0 -> 1
- net /vsys: track 49.8 -> 52.0 mm

Commit message: 3D model changes, added ETH passthrough and remodelled AA battery bracket
Parts:
- removed R17: 0R, Jumper:SolderJumper-2_P1.3mm_Open_Pad1.0x1.5mm
- removed U2: Mini360, voltage reg:Mini360_step-down
Connections:
- SW1 pad 1: Net-(SW1-A) -> /vsys
Routing:
- net Net-(U2-OUT+): track 27.1 -> 0.00 mm
- net /vsys: track 52.0 -> 69.8 mm
- net Net-(SW1-A): track 9.09 -> 0.00 mm
Changed lines of the file:
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@@
       (drillshape 0)
       (scaleselection 1)
-      (outputdirectory "../../cable_tester/pcb_gerber/")
+      (outputdirectory "pcb_gerber/")
     )
   )
@@
   (net 53 "Net-(J4-Pin_2)")
   (net 54 "unconnected-(SW1-C-Pad3)")
-  (net 55 "Net-(SW1-A)")
-  (net 56 "Net-(U2-OUT+)")
   (footprint "Connector_JST:JST_XH_B8B-XH-AM_1x08_P2.50mm_Vertical" (layer "F.Cu")
     (at 185.42 58.34 90)
@@
     (pad "" thru_hole oval (at 6.1 0) (size 2.2 3.5) (drill 1.5) (layers "*.Cu" "*.Mask"))
     (pad "1" thru_hole rect (at 0 0) (size 1.5 2.5) (drill 0.8) (layers "*.Cu" "*.Mask")
-      (net 55 "Net-(SW1-A)") (pinfunction "A") (pintype "passive"))
+      (net 11 "/vsys") (pinfunction "A") (pintype "passive"))
     (pad "2" thru_hole oval (at 2 0) (size 1.5 2.5) (drill 0.8) (layers "*.Cu" "*.Mask")
       (net 53 "Net-(J4-Pin_2)") (pinfunction "B") (pintype "passive"))
@@
     )
   )
-  (footprint "Jumper:SolderJumper-2_P1.3mm_Open_Pad1.0x1.5mm" (layer "F.Cu")
-    (at 174.61 88.9 180)
-    (descr "SMD Solder Jumper, 1x1.5mm Pads, 0.3mm gap, open")
-    (tags "solder jumper open")
-    (property "Sheetfile" "PCB.kicad_sch")
-    (property "Sheetname" "")
-    (property "ki_description" "Resistor")
-    (property "ki_keywords" "R res resistor")
-    (attr exclude_from_pos_files)
-    (fp_text reference "R17" (at 0 -1.8) (layer "F.SilkS") hide
-        (effects (font (size 1 1) (thickness 0.15)))
-    )
-    (fp_text value "0R" (at 0 -2.54) (layer "F.Fab")
-        (effects (font (size 1 1) (thickness 0.15)))
-    )
-    (fp_text user "Converter Connect" (at -0.65 2.54 unlocked) (layer "F.SilkS")
-        (effects (font (size 1 1) (thickness 0.15)))
-    )
-    (fp_line (start -1.4 -1) (end 1.4 -1)
-      (stroke (width 0.12) (type solid)) (layer "F.SilkS"))
-    (fp_line (start -1.4 1) (end -1.4 -1)
-      (stroke (width 0.12) (type solid)) (layer "F.SilkS"))
-    (fp_line (start 1.4 -1) (end 1.4 1)
-      (stroke (width 0.12) (type solid)) (layer "F.SilkS"))
-    (fp_line (start 1.4 1) (end -1.4 1)
-      (stroke (width 0.12) (type solid)) (layer "F.SilkS"))
-    (fp_line (start -1.65 -1.25) (end -1.65 1.25)
-      (stroke (width 0.05) (type solid)) (layer "F.CrtYd"))
-    (fp_line (start -1.65 -1.25) (end 1.65 -1.25)
-      (stroke (width 0.05) (type solid)) (layer "F.CrtYd"))
-    (fp_line (start 1.65 1.25) (end -1.65 1.25)
-      (stroke (width 0.05) (type solid)) (layer "F.CrtYd"))
-    (fp_line (start 1.65 1.25) (end 1.65 -1.25)
-      (stroke (width 0.05) (type solid)) (layer "F.CrtYd"))
-    (pad "1" smd rect (at -0.65 0 180) (size 1 1.5) (layers "F.Cu" "F.Mask")
-      (net 56 "Net-(U2-OUT+)") (pintype "passive"))
-    (pad "2" smd rect (at 0.65 0 180) (size 1 1.5) (layers "F.Cu" "F.Mask")
-      (net 11 "/vsys") (pintype "passive"))
-  )
   (footprint "Connector_JST:JST_XH_B8B-XH-AM_1x08_P2.50mm_Vertical" (layer "F.Cu")
     (at 195.58 58.34 90)
@@
     )
   )
-  (footprint "voltage reg:Mini360_step-down" (layer "F.Cu")
-    (at 190.5 94.49)
-    (property "Sheetfile" "PCB.kicad_sch")
-    (property "Sheetname" "")
-    (attr through_hole)
-    (fp_text reference "U2" (at 0 0.5) (layer "F.SilkS")
-        (effects (font (size 1 1) (thickness 0.15)))
-    )
-    (fp_text value "Mini360" (at 0 -0.5) (layer "F.Fab")
-        (effects (font (size 1 1) (thickness 0.15)))
-    )
-    (fp_line (start -8.75 -5.54) (end -8.75 5.53)
-      (stroke (width 0.15) (type solid)) (layer "F.SilkS"))
-    (fp_line (start -8.75 -5.54) (end 8.75 -5.54)
-      (stroke (width 0.15) (type solid)) (layer "F.SilkS"))
-    (fp_line (start 8.75 5.53) (end -8.75 5.53)
-      (stroke (width 0.15) (type solid)) (layer "F.SilkS"))
-    (fp_line (start 8.75 5.53) (end 8.75 -5.54)
-      (stroke (width 0.15) (type solid)) (layer "F.SilkS"))
-    (pad "1" thru_hole oval (at -7.62 -4.57) (size 2.5 2) (drill 0.762) (layers "*.Cu" "*.Mask")
-      (net 25 "GND") (pinfunction "IN-") (pintype "power_in"))
-    (pad "2" thru_hole oval (at -7.62 4.57) (size 2.5 2) (drill 0.762) (layers "*.Cu" "*.Mask")
-      (net 55 "Net-(SW1-A)") (pinfunction "IN+") (pintype "power_in"))
-    (pad "3" thru_hole oval (at 7.62 -4.57) (size 2.5 2) (drill 0.762) (layers "*.Cu" "*.Mask")
-      (net 25 "GND") (pinfunction "OUT-") (pintype "power_out"))
-    (pad "4" thru_hole oval (at 7.62 4.57) (size 2.5 2) (drill 0.762) (layers "*.Cu" "*.Mask")
-      (net 56 "Net-(U2-OUT+)") (pinfunction "OUT+") (pintype "power_out"))
-  )
   (footprint "Resistor_SMD:R_0805_2012Metric" (layer "F.Cu")
     (at 177.8 40.64)
@@
   (segment (start 153.765 96.115) (end 153.765 60.865) (width 0.25) (layer "B.Cu") (net 5))
   (segment (start 153.765 60.865) (end 161.29 53.34) (width 0.25) (layer "B.Cu") (net 5))
-  (segment (start 170.18 88.9) (end 173.96 88.9) (width 0.25) (layer "F.Cu") (net 11))
+  (segment (start 172.72 91.44) (end 170.18 88.9) (width 0.25) (layer "F.Cu") (net 11))
+  (segment (start 179.32 102.62) (end 172.72 96.02) (width 0.25) (layer "F.Cu") (net 11))
+  (segment (start 179.32 106.68) (end 179.32 102.62) (width 0.25) (layer "F.Cu") (net 11))
+  (segment (start 172.72 96.02) (end 172.72 91.44) (width 0.25) (layer "F.Cu") (net 11))
   (via (at 170.18 88.9) (size 0.8) (drill 0.4) (layers "F.Cu" "B.Cu") (net 11))
   (segment (start 170.18 52.314695) (end 163.585305 45.72) (width 0.25) (layer "B.Cu") (net 11))
@@
   (segment (start 175.3 96.52) (end 181.32 102.54) (width 0.25) (layer "B.Cu") (net 53))
   (segment (start 181.32 102.54) (end 181.32 106.68) (width 0.25) (layer "B.Cu") (net 53))
-  (segment (start 179.32 102.62) (end 182.88 99.06) (width 0.25) (layer "F.Cu") (net 55))
-  (segment (start 179.32 106.68) (end 179.32 102.62) (width 0.25) (layer "F.Cu") (net 55))
-  (segment (start 185.42 99.06) (end 175.26 88.9) (width 0.25) (layer "F.Cu") (net 56))
-  (segment (start 198.12 99.06) (end 185.42 99.06) (width 0.25) (layer "F.Cu") (net 56))
   (zone (net 25) (net_name "GND") (layers "F&B.Cu") (hatch edge 0.5)
     (connect_pads (clearance 0.5))
     (min_thickness 0.25) (filled_areas_thickness no)
-    (fill (thermal_gap 0.5) (thermal_bridge_width 0.5))
+    (fill yes (thermal_gap 0.5) (thermal_bridge_width 0.5))
     (polygon
       (pts
